Commit message: Add Navigation Stack and Move Base, TEB Local Planner

File: src/simulation/robot/urdf/gem.xacro (robot description, xacro)
@@ -90,4 +90,14 @@
     <dynamics damping="0.0" friction="0.0"/>
   </joint>
+  <transmission name="trans_${lr}_rotate">
+    <type>transmission_interface/SimpleTransmission</type>
+    <joint name="${lr}_rotate">
+      <hardwareInterface>hardware_interface/EffortJointInterface</hardwareInterface>
+    </joint>
+    <actuator name="motor_${lr}_rotate">
+      <hardwareInterface>hardware_interface/EffortJointInterface</hardwareInterface>
+      <mechanicalReduction>1</mechanicalReduction>
+    </actuator>
+  </transmission>
 </xacro:macro>
 	<!--<macro name="box_inertia" params="m x y z">
@@ -170,3 +180,11 @@
 		</plugin>
 	</gazebo>
+  <gazebo>
+    <plugin name="ground_truth" filename="libgazebo_ros_p3d.so">
+      <frameName>map</frameName>
+      <bodyName>base_link</bodyName>
+      <topicName>odom</topicName>
+      <updateRate>30.0</updateRate>
+    </plugin>
+  </gazebo>
 </robot>
